Commit message: Finish chapter_4 with FlexBE, partial chapter_5.

File: custom_ws/src/robot_description/urdf/mobile_manipulator.urdf.xacro (robot description, xacro)
@@ -6,3 +6,66 @@
   <xacro:arm_joint prefix="arm_base" parent="base_link" child="arm_base"
     originxyz="0.20 0.0 0.145" originrpy="0 0 0" axisxyz="0 0 1"/>
+  <!-- ######################### SENSORS ####################### -->
+  <link name="laser_link">
+    <visual>
+      <origin xyz="0.0 0.0 0.0" rpy="0.0 0.0 0.0"/>
+      <geometry>
+        <box size="0.05 0.05 0.05"/>
+      </geometry>
+    </visual>
+    <collision>
+      <origin xyz="0.0 0.0 0.0" rpy="0.0 0.0 0.0"/>
+      <geometry>
+        <box size="0.1 0.1 0.1"/>
+      </geometry>
+    </collision>
+    <inertial>
+      <origin xyz="0.0 0.0 0.0" rpy="0.0 0.0 0.0"/>
+      <mass value="1e-5"/>
+      <inertia ixx="1e-6" ixy="0.0" ixz="0.0" iyy="1e-6" iyz="0.0" izz="1e-6"/>
+    </inertial>
+  </link>
+  <joint name="laser_joint" type="fixed">
+    <origin xyz="0.35 0.0 0.115" rpy="0.0 0.0 0.0"/>
+    <parent link="base_link"/>
+    <child link="laser_link"/>
+    <axis xyz="0.0 1 0.0"/>
+  </joint>
+  <!-- Hokuyo Laser -->
+  <gazebo reference="laser_link">
+    <sensor type="ray" name="laser">
+      <pose>0 0 0 0 0 0</pose>
+      <visualize>true</visualize>
+      <update_rate>40</update_rate>
+      <ray>
+        <scan>
+          <horizontal>
+            <samples>720</samples>
+            <resolution>1</resolution>
+            <min_angle>-1.570796</min_angle>
+            <max_angle>1.570796</max_angle>
+          </horizontal>
+        </scan>
+        <range>
+          <min>0.1</min>
+          <max>30.0</max>
+          <resolution>0.01</resolution>
+        </range>
+        <noise>
+          <type>gaussian</type>
+          <!-- Noise parameters based on published spec for Hokuyo laser
+          achieving "+-30mm" accuracy at range < 10m.  A mean of 0.0m and
+          stddev of 0.01m will put 99.7% of samples within 0.03m of the true
+          reading. -->
+          <mean>0.0</mean>
+          <stddev>0.01</stddev>
+        </noise>
+      </ray>
+      <plugin name="gazebo_ros_head_hokuyo_controller"
+        filename="libgazebo_ros_laser.so">
+        <topicName>/scan</topicName>
+        <frameName>laser_link</frameName>
+      </plugin>
+    </sensor>
+  </gazebo>
 </robot>
