Commit message: FInish Chapter 5 and partial Chapter 6.

File: custom_ws/src/robot_description/urdf/gazebo_essentials_base.xacro (robot description, xacro)
@@ -1,6 +1,16 @@
 <?xml version="1.0"?>
 <robot xmlns:xacro="http://www.ros.org/wiki/xacro" name="gazebo_essentials_base">
+  gazebo_ros_control plugin with argument as namespace
+  <xacro:arg name="nsm" default="robot0"/>
+  <gazebo>
+    <plugin name="gazebo_ros_control" filename="libgazebo_ros_control.so">
+      <robotNamespace>/$(arg nsp)</robotNamespace>
+      <controlPeriod>0.001</controlPeriod>
+      <robotParam>/$(arg nsp)/robot_description</robotParam>
+      <legacyModeNS>false</legacyModeNS>
+    </plugin>
+  </gazebo>
   <!-- gazebo_ros_control plugin -->
-  <gazebo>
+  <!-- <gazebo>
     <plugin name="gazebo_ros_control" filename="libgazebo_ros_control.so">
       <robotNamespace>/</robotNamespace>
@@ -9,5 +19,5 @@
       <legacyModeNS>false</legacyModeNS>
     </plugin>
-  </gazebo>
+  </gazebo> -->
   <!-- Gazebo differential drive plugin -->
   <gazebo>
@@ -20,13 +30,14 @@
       <wheelSeparation>0.5</wheelSeparation>
       <wheelDiameter>0.2</wheelDiameter>
-      <wheelTorque>10</wheelTorque>
+      <wheelTorque>20</wheelTorque>
       <publishTf>1</publishTf>
-      <odometryFrame>map</odometryFrame>
+      <odometryFrame>odom</odometryFrame>
       <commandTopic>cmd_vel</commandTopic>
       <odometryTopic>odom</odometryTopic>
-      <robotBaseFrame>base_link</robotBaseFrame>
+      <robotBaseFrame>base_footprint</robotBaseFrame>
       <wheelAcceleration>2.8</wheelAcceleration>
       <publishWheelJointState>true</publishWheelJointState>
-      <publishWheelTF>false</publishWheelTF>
+      <publishWheelTF>true</publishWheelTF>
+      <publishOdom>true</publishOdom>
       <odometrySource>1</odometrySource>
       <rosDebugLevel>Debug</rosDebugLevel>

File: custom_ws/src/robot_description/urdf/mobile_manipulator.urdf.xacro (robot description, xacro)
@@ -37,10 +37,10 @@
       <pose>0 0 0 0 0 0</pose>
       <visualize>true</visualize>
-      <update_rate>40</update_rate>
+      <update_rate>5</update_rate>
       <ray>
         <scan>
           <horizontal>
             <samples>720</samples>
-            <resolution>1</resolution>
+            <resolution>2</resolution>
             <min_angle>-1.570796</min_angle>
             <max_angle>1.570796</max_angle>
@@ -49,16 +49,16 @@
         <range>
           <min>0.1</min>
-          <max>30.0</max>
-          <resolution>0.01</resolution>
+          <max>200.0</max>
+          <resolution>0.02</resolution>
         </range>
-        <noise>
+        <!-- <noise>
           <type>gaussian</type>
-          <!-- Noise parameters based on published spec for Hokuyo laser
+          Noise parameters based on published spec for Hokuyo laser
           achieving "+-30mm" accuracy at range < 10m.  A mean of 0.0m and
           stddev of 0.01m will put 99.7% of samples within 0.03m of the true
-          reading. -->
+          reading.
           <mean>0.0</mean>
           <stddev>0.01</stddev>
-        </noise>
+        </noise> -->
       </ray>
       <plugin name="gazebo_ros_head_hokuyo_controller"

File: custom_ws/src/robot_description/urdf/robot_base.urdf.xacro (robot description, xacro)
@@ -9,57 +9,64 @@
 <!-- Include gazebo_essentials_base xacro -->
 <xacro:include filename="$(find robot_description)/urdf/gazebo_essentials_base.xacro"/>
-  <link name="base_link">
-    <visual>
-      <origin xyz="0.0 0.0 0.0" rpy="1.5707963267949 0 3.14"/>
-      <geometry>
-        <mesh
-          filename="package://robot_description/meshes/robot_base.stl"
-          scale="1.0 1.0 1.0"/>
-      </geometry>
-      <material name="">
-        <color rgba="0.79216 0.81961 0.93333 1.0"/>
-      </material>
-    </visual>
-    <collision>
-      <origin xyz="0.0 0.0 0.0" rpy="1.5707963267949 0.0 3.14"/>
-      <geometry>
-        <mesh
-          filename="package://robot_description/meshes/robot_base.stl"
-          scale="1.0 1.0 1.0"/>
-      </geometry>
-    </collision>
-    <inertial>
-      <origin
-        xyz="0.0030946 4.78250032638821E-11 0.053305"
-        rpy="0.0 0.0 0.0"/>
-      <mass value="47.873"/>
-      <inertia
-        ixx="0.774276574699151"
-        ixy="-1.03781944357671E-10"
-        ixz="0.00763014265820928"
-        iyy="1.64933255189991"
-        iyz="1.09578155845563E-12"
-        izz="2.1239326987473"/>
-    </inertial>
-  </link>
+<link name="base_footprint">/</link>
+<joint name="base_joint" type="fixed" >
+  <parent link="base_footprint" />
+  <child link="base_link" />
+  <origin xyz="0.0 0.0 0.1" rpy="0.0 0.0 0.0" />
+  <axis xyz="0.0 1 0.0"/>
+</joint>
+<link name="base_link">
+  <visual>
+    <origin xyz="0.0 0.0 0.0" rpy="1.5707963267949 0 3.14"/>
+    <geometry>
+      <mesh
+        filename="package://robot_description/meshes/robot_base.stl"
+        scale="1.0 1.0 1.0"/>
+    </geometry>
+    <material name="">
+      <color rgba="0.79216 0.81961 0.93333 1.0"/>
+    </material>
+  </visual>
+  <collision>
+    <origin xyz="0.0 0.0 0.0" rpy="1.5707963267949 0.0 3.14"/>
+    <geometry>
+      <mesh
+        filename="package://robot_description/meshes/robot_base.stl"
+        scale="1.0 1.0 1.0"/>
+    </geometry>
+  </collision>
+  <inertial>
+    <origin
+      xyz="0.0030946 4.78250032638821E-11 0.053305"
+      rpy="0.0 0.0 0.0"/>
+    <mass value="47.873"/>
+    <inertia
+      ixx="0.774276574699151"
+      ixy="-1.03781944357671E-10"
+      ixz="0.00763014265820928"
+      iyy="1.64933255189991"
+      iyz="1.09578155845563E-12"
+      izz="2.1239326987473"/>
+  </inertial>
+</link>
 <!-- Robot wheel links -->
-  <xacro:robot_wheel prefix="front_left"/>
-  <xacro:robot_wheel prefix="front_right"/>
-  <xacro:robot_wheel prefix="rear_left"/>
-  <xacro:robot_wheel prefix="rear_right"/>
+<xacro:robot_wheel prefix="front_left"/>
+<xacro:robot_wheel prefix="front_right"/>
+<xacro:robot_wheel prefix="rear_left"/>
+<xacro:robot_wheel prefix="rear_right"/>
 <!-- Robot wheel joints -->
-  <xacro:wheel_joint prefix="front_left" origin="0.220 0.250 0"/>
-  <xacro:wheel_joint prefix="front_right" origin="0.220 -0.250 0"/>
-  <xacro:wheel_joint prefix="rear_left" origin="-0.220 0.250 0"/>
-  <xacro:wheel_joint prefix="rear_right" origin="-0.220 -0.250 0"/>
+<xacro:wheel_joint prefix="front_left" origin="0.220 0.250 0"/>
+<xacro:wheel_joint prefix="front_right" origin="0.220 -0.250 0"/>
+<xacro:wheel_joint prefix="rear_left" origin="-0.220 0.250 0"/>
+<xacro:wheel_joint prefix="rear_right" origin="-0.220 -0.250 0"/>
 <!-- Wheels transmission elements -->
-  <xacro:base_transmission prefix="front_left"/>
-  <xacro:base_transmission prefix="front_right"/>
-  <xacro:base_transmission prefix="rear_left"/>
-  <xacro:base_transmission prefix="rear_right"/>
+<xacro:base_transmission prefix="front_left"/>
+<xacro:base_transmission prefix="front_right"/>
+<xacro:base_transmission prefix="rear_left"/>
+<xacro:base_transmission prefix="rear_right"/>
 <!-- Wheel friction macro for gazebo -->
-  <xacro:wheel_friction prefix="front_left"/>
-  <xacro:wheel_friction prefix="front_right"/>
-  <xacro:wheel_friction prefix="rear_left"/>
-  <xacro:wheel_friction prefix="rear_right"/>
+<xacro:wheel_friction prefix="front_left"/>
+<xacro:wheel_friction prefix="front_right"/>
+<xacro:wheel_friction prefix="rear_left"/>
+<xacro:wheel_friction prefix="rear_right"/>
 </robot>
